File: STM32-USBc/STM32-USBc.kicad_sch (KiCad schematic)
At the start: 19 parts, among them J1 Conn_01x04_Pin, P1 USB_C_Plug_USB2.0, SW1 SW_SPDT, U1 STM32F103C8T6, Y3 16MHz

Commit message: improve placements
Parts:
- added C12, C13: 22u, symbol Device:C
- added D1: LED, symbol Device:LED
- added J2, J3: Conn_01x04_Pin, symbol Connector:Conn_01x04_Pin
- added R3, R4, R5: 1k5, symbol Device:R
- added U2: AMS1117-3.3, Package_TO_SOT_SMD:SOT-223-3_TabPin2, symbol Regulator_Linear:AMS1117-3.3
Connections:
- net +3.3V: now also C13.1, D1.2 (A), J2.1 (Pin_1), J3.1 (Pin_1), R4.1, R5.1, U2.2 (VO)
- net GND: now also C12.2, C13.2, J2.4 (Pin_4), J3.4 (Pin_4), R3.2, U2.1 (GND)
- net VBUS: now also C12.1, U2.3 (VI)
- net I2C2_SCL: now reaches U1.21 (PB10)
- net I2C2_SCL: now also J3.2 (Pin_2), R4.2
- net I2C2_SDA: now reaches U1.22 (PB11)
- net I2C2_SDA: now also J3.3 (Pin_3), R5.2
- net USART1_TX: now reaches U1.42 (PB6)
- net USART1_TX: now also J2.2 (Pin_2)
- net USART1_RX: now reaches U1.43 (PB7)
- net USART1_RX: now also J2.3 (Pin_3)
- new net PWR_LED_K: D1.1 (K), R3.1
- no-connect marks 3 -> 30
Other:
- note added: "STM32-UBS-C (experimental)"
- title: (none) -> STM32-USB-C
- moved on the sheet: C1, C10, C11, C2, C3, C4, C5, C6, C7, C8, C9, FB1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
