File: STM32-USBc/STM32-USBc.kicad_sch (KiCad schematic)
At the start: 28 parts, among them J1 Conn_01x04_Pin, J2 Conn_01x04_Pin, J3 Conn_01x04_Pin, P1 USB_C_Plug_USB2.0, SW1 SW_SPDT, U1 STM32F103C8T6, U2 AMS1117-3.3, Y3 16MHz

Commit message: assign footprints
Parts:
- C1: renamed from C12; footprint (none) -> Capacitor_SMD:C_0805_2012Metric
- C10: renamed from C8; footprint (none) -> Capacitor_SMD:C_0402_1005Metric
- C11: renamed from C9; footprint (none) -> Capacitor_SMD:C_0402_1005Metric
- C12: renamed from C10; footprint (none) -> Capacitor_SMD:C_0402_1005Metric
- C13: renamed from C11; footprint (none) -> Capacitor_SMD:C_0402_1005Metric
- C2: renamed from C13; footprint (none) -> Capacitor_SMD:C_0805_2012Metric
- C3: renamed from C1; footprint (none) -> Capacitor_SMD:C_0402_1005Metric
- C4: renamed from C2; footprint (none) -> Capacitor_SMD:C_0402_1005Metric
- C5: renamed from C3; footprint (none) -> Capacitor_SMD:C_0402_1005Metric
- C6: renamed from C4; footprint (none) -> Capacitor_SMD:C_0402_1005Metric
- C7: renamed from C5; footprint (none) -> Capacitor_SMD:C_0603_1608Metric
- C8: renamed from C6; footprint (none) -> Capacitor_SMD:C_0603_1608Metric
- C9: renamed from C7; footprint (none) -> Capacitor_SMD:C_0402_1005Metric
- D1: footprint (none) -> LED_SMD:LED_0603_1608Metric
- FB1: footprint (none) -> Inductor_SMD:L_0603_1608Metric
- J1, J2, J3: footprint (none) -> Connector_PinSocket_2.54mm:PinSocket_1x04_P2.54mm_Vertical
- P1: footprint (none) -> Connector_USB:USB_C_Receptacle_Molex_105450-0101
- R1: renamed from R3; footprint (none) -> Resistor_SMD:R_0402_1005Metric
- R2: renamed from R1; footprint (none) -> Resistor_SMD:R_0402_1005Metric
- R3: renamed from R2; footprint (none) -> Resistor_SMD:R_0402_1005Metric
- R4, R5: footprint (none) -> Resistor_SMD:R_0402_1005Metric
- SW1: footprint (none) -> Button_Switch_THT:SW_E-Switch_EG1224_SPDT_Angled
- Y3: footprint (none) -> Crystal:Crystal_SMD_3225-4Pin_3.2x2.5mm
Changed lines of the file:
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@@
 	(wire
 		(pts
+			(xy 241.3 66.04) (xy 247.65 66.04)
+		)
+		(stroke
+			(width 0)
+			(type default)
+		)
+	)
+	(wire
+		(pts
 			(xy 132.08 149.86) (xy 135.89 149.86)
 		)
@@
 	(wire
 		(pts
-			(xy 243.84 66.04) (xy 247.65 66.04)
-		)
-		(stroke
-			(width 0)
-			(type default)
-		)
-	)
-	(wire
-		(pts
 			(xy 91.44 52.07) (xy 91.44 48.26)
 		)
@@
 			)
 		)
-		(property "Footprint" ""
+		(property "Footprint" "Inductor_SMD:L_0603_1608Metric"
 			(at 229.87 30.988 90)
 			(effects
@@
 			)
 		)
-		(property "Footprint" ""
+		(property "Footprint" "Connector_PinSocket_2.54mm:PinSocket_1x04_P2.54mm_Vertical"
 			(at 127 116.84 0)
 			(effects
@@
 		(dnp no)
 		(fields_autoplaced yes)
-		(property "Reference" "C7"
+		(property "Reference" "C9"
 			(at 223.52 33.0199 0)
 			(effects
@@
 			)
 		)
-		(property "Footprint" ""
+		(property "Footprint" "Capacitor_SMD:C_0402_1005Metric"
 			(at 220.6752 38.1 0)
 			(effects
@@
 			(project "STM32-USBc"
 				(path "/cbd5a7da-407b-4de2-bd9e-9cdebe4da750"
-					(reference "C7")
+					(reference "C9")
 					(unit 1)
 				)
@@
 		(dnp no)
 		(fields_autoplaced yes)
-		(property "Reference" "C5"
+		(property "Reference" "C7"
 			(at 127 34.2899 0)
 			(effects
@@
 			)
 		)
-		(property "Footprint" ""
+		(property "Footprint" "Capacitor_SMD:C_0603_1608Metric"
 			(at 124.1552 39.37 0)
 			(effects
@@
 			(project "STM32-USBc"
 				(path "/cbd5a7da-407b-4de2-bd9e-9cdebe4da750"
-					(reference "C5")
+					(reference "C7")
 					(unit 1)
 				)
@@
 			)
 		)
-		(property "Footprint" ""
+		(property "Footprint" "Resistor_SMD:R_0402_1005Metric"
 			(at 141.732 138.43 90)
 			(effects
@@
 			)
 		)
-		(property "Footprint" ""
+		(property "Footprint" "Button_Switch_THT:SW_E-Switch_EG1224_SPDT_Angled"
 			(at 151.13 55.88 0)
 			(effects
@@
 			)
 		)
-		(property "Footprint" ""
+		(property "Footprint" "Connector_USB:USB_C_Receptacle_Molex_105450-0101"
 			(at 261.62 81.28 0)
 			(effects
@@
 		(dnp no)
 		(fields_autoplaced yes)
-		(property "Reference" "C10"
+		(property "Reference" "C12"
 			(at 120.65 95.2499 0)
 			(effects
@@
 			)
 		)
-		(property "Footprint" ""
+		(property "Footprint" "Capacitor_SMD:C_0402_1005Metric"
 			(at 117.8052 100.33 0)
 			(effects
@@
 			(project "STM32-USBc"
 				(path "/cbd5a7da-407b-4de2-bd9e-9cdebe4da750"
-					(reference "C10")
+					(reference "C12")
 					(unit 1)
 				)
@@
 			)
 		)
-		(property "Footprint" ""
+		(property "Footprint" "Connector_PinSocket_2.54mm:PinSocket_1x04_P2.54mm_Vertical"
 			(at 127 144.78 0)
 			(effects
@@
 		(dnp no)
 		(fields_autoplaced yes)
-		(property "Reference" "C2"
+		(property "Reference" "C4"
 			(at 162.56 34.2899 0)
 			(effects
@@
 			)
 		)
-		(property "Footprint" ""
+		(property "Footprint" "Capacitor_SMD:C_0402_1005Metric"
 			(at 159.7152 39.37 0)
 			(effects
@@
 			(project "STM32-USBc"
 				(path "/cbd5a7da-407b-4de2-bd9e-9cdebe4da750"
-					(reference "C2")
+					(reference "C4")
 					(unit 1)
 				)
@@
 			)
 		)
-		(property "Footprint" ""
+		(property "Footprint" "LED_SMD:LED_0603_1608Metric"
 			(at 80.01 48.26 0)
 			(effects
@@
 		(dnp no)
 		(fields_autoplaced yes)
-		(property "Reference" "C8"
+		(property "Reference" "C10"
 			(at 243.84 33.0199 0)
 			(effects
@@
 			)
 		)
-		(property "Footprint" ""
+		(property "Footprint" "Capacitor_SMD:C_0402_1005Metric"
 			(at 240.9952 38.1 0)
 			(effects
@@
 			(project "STM32-USBc"
 				(path "/cbd5a7da-407b-4de2-bd9e-9cdebe4da750"
-					(reference "C8")
+					(reference "C10")
 					(unit 1)
 				)
@@
 	(symbol
 		(lib_id "power:PWR_FLAG")
-		(at 243.84 66.04 0)
+		(at 241.3 66.04 0)
 		(unit 1)
 		(exclude_from_sim no)
@@
 		(fields_autoplaced yes)
 		(property "Reference" "#FLG02"
-			(at 243.84 64.135 0)
+			(at 241.3 64.135 0)
 			(effects
 				(font
@@
 		)
 		(property "Value" "PWR_FLAG"
-			(at 243.84 60.96 0)
+			(at 241.3 60.96 0)
 			(effects
 				(font
@@
 		)
 		(property "Footprint" ""
-			(at 243.84 66.04 0)
+			(at 241.3 66.04 0)
 			(effects
 				(font
@@
 		)
 		(property "Datasheet" "~"
-			(at 243.84 66.04 0)
+			(at 241.3 66.04 0)
 			(effects
 				(font
@@
 		)
 		(property "Description" "Special symbol for telling ERC where power comes from"
-			(at 243.84 66.04 0)
+			(at 241.3 66.04 0)
 			(effects
 				(font
@@
 			)
 		)
-		(property "Footprint" ""
+		(property "Footprint" "Connector_PinSocket_2.54mm:PinSocket_1x04_P2.54mm_Vertical"
 			(at 241.3 107.95 0)
 			(effects
@@
 		(dnp no)
 		(fields_autoplaced yes)
-		(property "Reference" "C3"
+		(property "Reference" "C5"
 			(at 149.86 34.2899 0)
 			(effects
@@
 			)
 		)
-		(property "Footprint" ""
+		(property "Footprint" "Capacitor_SMD:C_0402_1005Metric"
 			(at 147.0152 39.37 0)
 			(effects
@@
 			(project "STM32-USBc"
 				(path "/cbd5a7da-407b-4de2-bd9e-9cdebe4da750"
-					(reference "C3")
+					(reference "C5")
 					(unit 1)
 				)
@@
 		(dnp no)
 		(fields_autoplaced yes)
-		(property "Reference" "C1"
+		(property "Reference" "C3"
 			(at 173.99 34.2899 0)
 			(effects
@@
 			)
 		)
-		(property "Footprint" ""
+		(property "Footprint" "Capacitor_SMD:C_0402_1005Metric"
 			(at 171.1452 39.37 0)
 			(effects
@@
 			(project "STM32-USBc"
 				(path "/cbd5a7da-407b-4de2-bd9e-9cdebe4da750"
-					(reference "C1")
+					(reference "C3")
 					(unit 1)
 				)
@@
 		(dnp no)
 		(fields_autoplaced yes)
-		(property "Reference" "C4"
+		(property "Reference" "C6"
 			(at 138.43 34.2899 0)
 			(effects
@@
 			)
 		)
-		(property "Footprint" ""
+		(property "Footprint" "Capacitor_SMD:C_0402_1005Metric"
 			(at 135.5852 39.37 0)
 			(effects
@@
 			(project "STM32-USBc"
 				(path "/cbd5a7da-407b-4de2-bd9e-9cdebe4da750"
-					(reference "C4")
+					(reference "C6")
 					(unit 1)
 				)
@@
 			)
 		)
-		(property "Footprint" ""
+		(property "Footprint" "Crystal:Crystal_SMD_3225-4Pin_3.2x2.5mm"
 			(at 128.27 83.82 0)
 			(effects
@@
 		(dnp no)
 		(fields_autoplaced yes)
-		(property "Reference" "C9"
+		(property "Reference" "C11"
 			(at 127 57.1499 0)
 			(effects
@@
 			)
 		)
-		(property "Footprint" ""
+		(property "Footprint" "Capacitor_SMD:C_0402_1005Metric"
 			(at 124.1552 62.23 0)
 			(effects
@@
 			(project "STM32-USBc"
 				(path "/cbd5a7da-407b-4de2-bd9e-9cdebe4da750"
-					(reference "C9")
+					(reference "C11")
 					(unit 1)
 				)
@@
 			)
 		)
-		(property "Footprint" ""
+		(property "Footprint" "Resistor_SMD:R_0402_1005Metric"
 			(at 151.892 138.43 90)
 			(effects
@@
 		(dnp no)
 		(fields_autoplaced yes)
-		(property "Reference" "C12"
+		(property "Reference" "C1"
 			(at 31.75 54.6099 0)
 			(effects
@@
 			)
 		)
-		(property "Footprint" ""
+		(property "Footprint" "Capacitor_SMD:C_0805_2012Metric"
 			(at 28.9052 59.69 0)
 			(effects
@@
 			(project ""
 				(path "/cbd5a7da-407b-4de2-bd9e-9cdebe4da750"
-					(reference "C12")
+					(reference "C1")
 					(unit 1)
 				)
@@
 		(dnp no)
 		(fields_autoplaced yes)
-		(property "Reference" "C6"
+		(property "Reference" "C8"
 			(at 210.82 33.0199 0)
 			(effects
@@
 			)
 		)
-		(property "Footprint" ""
+		(property "Footprint" "Capacitor_SMD:C_0603_1608Metric"
 			(at 207.9752 38.1 0)
 			(effects
@@
 			(project "STM32-USBc"
 				(path "/cbd5a7da-407b-4de2-bd9e-9cdebe4da750"
-					(reference "C6")
+					(reference "C8")
 					(unit 1)
 				)
@@
 		(dnp no)
 		(fields_autoplaced yes)
-		(property "Reference" "C11"
+		(property "Reference" "C13"
 			(at 147.32 95.2499 0)
 			(effects
@@
 			)
 		)
-		(property "Footprint" ""
+		(property "Footprint" "Capacitor_SMD:C_0402_1005Metric"
 			(at 144.4752 100.33 0)
 			(effects
@@
 			(project "STM32-USBc"
 				(path "/cbd5a7da-407b-4de2-bd9e-9cdebe4da750"
-					(reference "C11")
+					(reference "C13")
 					(unit 1)
 				)
@@
 		(dnp no)
 		(fields_autoplaced yes)
-		(property "Reference" "C13"
+		(property "Reference" "C2"
 			(at 66.04 54.6099 0)
 			(effects
@@
 			)
 		)
-		(property "Footprint" ""
+		(property "Footprint" "Capacitor_SMD:C_0805_2012Metric"
 			(at 63.1952 59.69 0)
 			(effects
@@
 			(project "STM32-USBc"
 				(path "/cbd5a7da-407b-4de2-bd9e-9cdebe4da750"
-					(reference "C13")
+					(reference "C2")
 					(unit 1)
 				)
@@
 		(on_board yes)
 		(dnp no)
-		(property "Reference" "R1"
+		(property "Reference" "R2"
 			(at 165.1 53.594 90)
 			(effects
@@
 			)
 		)
-		(property "Footprint" ""
+		(property "Footprint" "Resistor_SMD:R_0402_1005Metric"
 			(at 165.1 57.658 90)
 			(effects
@@
 			(project "STM32-USBc"
 				(path "/cbd5a7da-407b-4de2-bd9e-9cdebe4da750"
-					(reference "R1")
+					(reference "R2")
 					(unit 1)
 				)
@@
 		(on_board yes)
 		(dnp no)
-		(property "Reference" "R3"
+		(property "Reference" "R1"
 			(at 93.98 54.6099 0)
 			(effects
@@
 			)
 		)
-		(property "Footprint" ""
+		(property "Footprint" "Resistor_SMD:R_0402_1005Metric"
 			(at 89.662 55.88 90)
 			(effects
@@
 			(project ""
 				(path "/cbd5a7da-407b-4de2-bd9e-9cdebe4da750"
-					(reference "R3")
+					(reference "R1")
 					(unit 1)
 				)
@@
 		(dnp no)
 		(fields_autoplaced yes)
-		(property "Reference" "R2"
+		(property "Reference" "R3"
 			(at 232.41 69.8499 0)
 			(effects
@@
 			)
 		)
-		(property "Footprint" ""
+		(property "Footprint" "Resistor_SMD:R_0402_1005Metric"
 			(at 228.092 71.12 90)
 			(effects
@@
 			(project "STM32-USBc"
 				(path "/cbd5a7da-407b-4de2-bd9e-9cdebe4da750"
-					(reference "R2")
+					(reference "R3")
 					(unit 1)
 				)
