File: STM32-USBb/STM32-USBb.kicad_sch (KiCad schematic)
At the start: 32 parts, among them J1 Conn_01x04_Pin, J2 Conn_01x04_Pin, J3 Conn_01x04_Pin, J4 USB_B_Micro, SW1 SW_SPDT, U1 STM32F103C8T6, U2 AMS1117-3.3, Y3 16MHz

Commit message: changing for usb b
Parts:
- J4: footprint Connector_USB:USB_Micro-B_Wuerth_629105150521 -> (none)
Changed lines of the file:
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@@
 		)
 		(instances
-			(project "STM32-USBc"
+			(project "STM32-USBb"
 				(path "/cbd5a7da-407b-4de2-bd9e-9cdebe4da750"
 					(reference "#PWR011")
@@
 		)
 		(instances
-			(project "STM32-USBc"
+			(project "STM32-USBb"
 				(path "/cbd5a7da-407b-4de2-bd9e-9cdebe4da750"
 					(reference "FB1")
@@
 		)
 		(instances
-			(project "STM32-USBc"
+			(project "STM32-USBb"
 				(path "/cbd5a7da-407b-4de2-bd9e-9cdebe4da750"
 					(reference "J2")
@@
 		)
 		(instances
-			(project "STM32-USBc"
+			(project "STM32-USBb"
 				(path "/cbd5a7da-407b-4de2-bd9e-9cdebe4da750"
 					(reference "C9")
@@
 		)
 		(instances
-			(project "STM32-USBc"
+			(project "STM32-USBb"
 				(path "/cbd5a7da-407b-4de2-bd9e-9cdebe4da750"
 					(reference "C7")
@@
 		)
 		(instances
-			(project "STM32-USBc"
+			(project "STM32-USBb"
 				(path "/cbd5a7da-407b-4de2-bd9e-9cdebe4da750"
 					(reference "SW1")
@@
 		)
 		(instances
-			(project "STM32-USBc"
+			(project "STM32-USBb"
 				(path "/cbd5a7da-407b-4de2-bd9e-9cdebe4da750"
 					(reference "#PWR015")
@@
 		)
 		(instances
-			(project "STM32-USBc"
+			(project "STM32-USBb"
 				(path "/cbd5a7da-407b-4de2-bd9e-9cdebe4da750"
 					(reference "#PWR07")
@@
 		)
 		(instances
-			(project "STM32-USBc"
+			(project "STM32-USBb"
 				(path "/cbd5a7da-407b-4de2-bd9e-9cdebe4da750"
 					(reference "#PWR08")
@@
 		)
 		(instances
-			(project "STM32-USBc"
+			(project "STM32-USBb"
 				(path "/cbd5a7da-407b-4de2-bd9e-9cdebe4da750"
 					(reference "C12")
@@
 		)
 		(instances
-			(project "STM32-USBc"
+			(project "STM32-USBb"
 				(path "/cbd5a7da-407b-4de2-bd9e-9cdebe4da750"
 					(reference "J3")
@@
 		)
 		(instances
-			(project "STM32-USBc"
+			(project "STM32-USBb"
 				(path "/cbd5a7da-407b-4de2-bd9e-9cdebe4da750"
 					(reference "C4")
@@
 			)
 		)
-		(property "Footprint" "Connector_USB:USB_Micro-B_Wuerth_629105150521"
+		(property "Footprint" ""
 			(at 264.16 77.47 0)
 			(effects
@@
 		)
 		(instances
-			(project "STM32-USBc"
+			(project "STM32-USBb"
 				(path "/cbd5a7da-407b-4de2-bd9e-9cdebe4da750"
 					(reference "C10")
@@
 		)
 		(instances
-			(project "STM32-USBc"
+			(project "STM32-USBb"
 				(path "/cbd5a7da-407b-4de2-bd9e-9cdebe4da750"
 					(reference "H2")
@@
 		)
 		(instances
-			(project "STM32-USBc"
+			(project "STM32-USBb"
 				(path "/cbd5a7da-407b-4de2-bd9e-9cdebe4da750"
 					(reference "J1")
@@
 		)
 		(instances
-			(project "STM32-USBc"
+			(project "STM32-USBb"
 				(path "/cbd5a7da-407b-4de2-bd9e-9cdebe4da750"
 					(reference "#PWR023")
@@
 		)
 		(instances
-			(project "STM32-USBc"
+			(project "STM32-USBb"
 				(path "/cbd5a7da-407b-4de2-bd9e-9cdebe4da750"
 					(reference "C5")
@@
 		)
 		(instances
-			(project "STM32-USBc"
+			(project "STM32-USBb"
 				(path "/cbd5a7da-407b-4de2-bd9e-9cdebe4da750"
 					(reference "#PWR013")
@@
 		)
 		(instances
-			(project "STM32-USBc"
+			(project "STM32-USBb"
 				(path "/cbd5a7da-407b-4de2-bd9e-9cdebe4da750"
 					(reference "C3")
@@
 		)
 		(instances
-			(project "STM32-USBc"
+			(project "STM32-USBb"
 				(path "/cbd5a7da-407b-4de2-bd9e-9cdebe4da750"
 					(reference "C6")
@@
 		)
 		(instances
-			(project "STM32-USBc"
+			(project "STM32-USBb"
 				(path "/cbd5a7da-407b-4de2-bd9e-9cdebe4da750"
 					(reference "Y3")
@@
 		)
 		(instances
-			(project "STM32-USBc"
+			(project "STM32-USBb"
 				(path "/cbd5a7da-407b-4de2-bd9e-9cdebe4da750"
 					(reference "#PWR03")
@@
 		)
 		(instances
-			(project "STM32-USBc"
+			(project "STM32-USBb"
 				(path "/cbd5a7da-407b-4de2-bd9e-9cdebe4da750"
 					(reference "H4")
@@
 		)
 		(instances
-			(project "STM32-USBc"
+			(project "STM32-USBb"
 				(path "/cbd5a7da-407b-4de2-bd9e-9cdebe4da750"
 					(reference "C11")
@@
 		)
 		(instances
-			(project "STM32-USBc"
+			(project "STM32-USBb"
 				(path "/cbd5a7da-407b-4de2-bd9e-9cdebe4da750"
 					(reference "H3")
@@
 		)
 		(instances
-			(project "STM32-USBc"
+			(project "STM32-USBb"
 				(path "/cbd5a7da-407b-4de2-bd9e-9cdebe4da750"
 					(reference "#PWR022")
@@
 		)
 		(instances
-			(project "STM32-USBc"
+			(project "STM32-USBb"
 				(path "/cbd5a7da-407b-4de2-bd9e-9cdebe4da750"
 					(reference "#PWR012")
@@
 		)
 		(instances
-			(project "STM32-USBc"
+			(project "STM32-USBb"
 				(path "/cbd5a7da-407b-4de2-bd9e-9cdebe4da750"
 					(reference "#PWR010")
@@
 		)
 		(instances
-			(project "STM32-USBc"
+			(project "STM32-USBb"
 				(path "/cbd5a7da-407b-4de2-bd9e-9cdebe4da750"
 					(reference "#PWR02")
@@
 		)
 		(instances
-			(project "STM32-USBc"
+			(project "STM32-USBb"
 				(path "/cbd5a7da-407b-4de2-bd9e-9cdebe4da750"
 					(reference "R5")
@@
 		)
 		(instances
-			(project "STM32-USBc"
+			(project "STM32-USBb"
 				(path "/cbd5a7da-407b-4de2-bd9e-9cdebe4da750"
 					(reference "#PWR04")
@@
 		)
 		(instances
-			(project "STM32-USBc"
+			(project "STM32-USBb"
 				(path "/cbd5a7da-407b-4de2-bd9e-9cdebe4da750"
 					(reference "C8")
@@
 		)
 		(instances
-			(project "STM32-USBc"
+			(project "STM32-USBb"
 				(path "/cbd5a7da-407b-4de2-bd9e-9cdebe4da750"
 					(reference "#PWR05")
@@
 		)
 		(instances
-			(project "STM32-USBc"
+			(project "STM32-USBb"
 				(path "/cbd5a7da-407b-4de2-bd9e-9cdebe4da750"
 					(reference "#PWR021")
@@
 		)
 		(instances
-			(project "STM32-USBc"
+			(project "STM32-USBb"
 				(path "/cbd5a7da-407b-4de2-bd9e-9cdebe4da750"
 					(reference "#PWR09")
@@
 		)
 		(instances
-			(project "STM32-USBc"
+			(project "STM32-USBb"
 				(path "/cbd5a7da-407b-4de2-bd9e-9cdebe4da750"
 					(reference "C13")
@@
 		)
 		(instances
-			(project "STM32-USBc"
+			(project "STM32-USBb"
 				(path "/cbd5a7da-407b-4de2-bd9e-9cdebe4da750"
 					(reference "#PWR06")
@@
 		)
 		(instances
-			(project "STM32-USBc"
+			(project "STM32-USBb"
 				(path "/cbd5a7da-407b-4de2-bd9e-9cdebe4da750"
 					(reference "C2")
@@
 		)
 		(instances
-			(project "STM32-USBc"
+			(project "STM32-USBb"
 				(path "/cbd5a7da-407b-4de2-bd9e-9cdebe4da750"
 					(reference "R2")
@@
 		)
 		(instances
-			(project "STM32-USBc"
+			(project "STM32-USBb"
 				(path "/cbd5a7da-407b-4de2-bd9e-9cdebe4da750"
 					(reference "U1")
@@
 		)
 		(instances
-			(project "STM32-USBc"
+			(project "STM32-USBb"
 				(path "/cbd5a7da-407b-4de2-bd9e-9cdebe4da750"
 					(reference "R3")
@@
 		)
 		(instances
-			(project "STM32-USBc"
+			(project "STM32-USBb"
 				(path "/cbd5a7da-407b-4de2-bd9e-9cdebe4da750"
 					(reference "#PWR014")

Commit message: add previews
Other:
- title: STM32-USB-C -> STM32-USB-B
Changed lines of the file:
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@@
 	(paper "A4")
 	(title_block
-		(title "STM32-USB-C")
+		(title "STM32-USB-B")
 		(date "2026-02-21")
 		(rev "1.0")
